Commit message: homework finito

File: arm_description/urdf/arm.urdf.xacro (robot description, xacro)
@@ -10,4 +10,10 @@
     <color rgba="1 1 1 1"/>
   </material>
+  <link name="world"/>
+  <joint name="base_link_joint" type="fixed">
+      <origin rpy="0.0 0 0" xyz="0 0 0"/>
+      <parent link="world"/>
+      <child link="base_link"/>
+  </joint>
  <link name="base_link">
     <visual>
